File: hardware/stm32mp151aab3/CPU.sch (KiCad schematic (older format))
At the start: 0 parts

Commit message: update
Parts:
- added C? (x3): 100n, Capacitor_SMD:C_0805_2012Metric, symbol Device:C_Small
- added D?: D_Small, symbol Device:D_Small
- added FB?: Ferrite_Bead_Small, symbol Device:Ferrite_Bead_Small
- added R?: 3k, Resistor_SMD:R_0805_2012Metric, symbol Device:R_Small
- added R?: 10k, Resistor_SMD:R_0805_2012Metric, symbol Device:R_Small
- added U? (x2): STM32MP151AAB3, symbol stm32mp151:STM32MP151AAB3
Connections:
- new net: C?.1, FB?.1, U?.M4 (VDDA)
- new net: C?.1, U?.N3 (VREF+)
- new net: R?.1, U?.V16 (USB_RREF)
- new net CPU_BOOT0: U?.K1 (BOOT0)
- new net CPU_BOOT1: U?.K4 (BOOT1)
- new net CPU_BOOT2: U?.L2 (BOOT2)
- new net CPU_JTDI: U?.D13 (JTDI)
- new net CPU_JTMS-SWDCLK: U?.D16 (JTCK-SWCLK)
- new net CPU_JTMS-SWDIO: U?.D15 (JTMS-SWDIO)
- new net CPU_JTMS-TRACESW0: U?.D14 (JTDO-TRACESWO)
- new net CPU_NJRST: U?.D12 (NJTRST)
- new net CPU_NRST: C?.1, D?.1 (K), U?.J1 (NRST), U?.J2 (NRST_CORE)
- new net GND: C?.2, C?.2, C?.2, R?.2, U?.A1 (VSS), U?.A19 (VSS), U?.B2 (VSS), U?.B6 (VSS), U?.C12 (VSS), U?.C13 (VSS), U?.C14 (VSS), U?.C15 (VSS), U?.C16 (VSS), U?.C17 (VSS), U?.C3 (VSS), U?.D1 (VSS), U?.D4 (VSS), U?.D5 (VSS), U?.D8 (VSS), U?.E10 (VSS), U?.E12 (VSS), U?.E14 (VSS), U?.E16 (VSS), U?.E2 (VSS), U?.E4 (VSS), U?.E5 (VSS), U?.E6 (VSS), U?.E8 (VSS), U?.F11 (VSS), U?.F13 (VSS_PLL2), U?.F15 (VSS), U?.F5 (VSS), U?.F7 (VSS), U?.F9 (VSS), U?.G10 (VSS), U?.G12 (VSS), U?.G14 (VSS), U?.G2 (VSS), U?.G4 (VSS), U?.G6 (VSS), U?.G8 (VSS), U?.H11 (VSS), U?.H13 (VSS), U?.H15 (VSS), U?.H5 (VSS), U?.H7 (VSS), U?.H9 (VSS), U?.J10 (VSS), U?.J12 (VSS), U?.J14 (VSS), U?.J3 (VSS), U?.J4 (VSS_PLL), U?.J6 (VSS), U?.J8 (VSS), U?.K11 (VSS), U?.K13 (VSS), U?.K15 (VSS), U?.K2 (VSS), U?.K5 (VSS), U?.K7 (VSS), U?.K9 (VSS), U?.L10 (VSS), U?.L12 (VSS), U?.L14 (VSS), U?.L4 (VSS_ANA), U?.L6 (VSS), U?.L8 (VSS), U?.M11 (VSS), U?.M13 (VSS), U?.M15 (VSS), U?.M3 (VREF-), U?.M5 (VSS), U?.M7 (VSS), U?.M9 (VSS), U?.N10 (VSS), U?.N12 (VSS), U?.N14 (VSS), U?.N4 (VSSA), U?.N6 (VSS), U?.N8 (VSS), U?.P11 (VSS), U?.P13 (VSS), U?.P15 (VSS), U?.P5 (VSSA), U?.P7 (VSS), U?.P9 (VSS), U?.R10 (VSS), U?.R12 (VSS), U?.R14 (VSS), U?.R16 (VSS), U?.R2 (VSS), U?.R5 (VSSA), U?.R6 (VSS), U?.R8 (VSS), U?.T4 (VSS), U?.U13 (VSS_USBHS), U?.U14 (VSS_USBHS), U?.U17 (VSS), U?.U3 (VSS), U?.U6 (VSS), U?.U8 (VSS), U?.V12 (VSS_USBHS), U?.V15 (VSS_USBHS), U?.W1 (VSS), U?.W19 (VSS)
- new net PWR_LP: U?.P1 (PWR_LP)
- new net PWR_ON: R?.1, U?.L1 (PWR_ON)
- new net PWR_ONRST: D?.2 (A), R?.2
- new net USB_DM1: U?.W14 (USB_DM1)
- new net USB_DM2: U?.V13 (USB_DM2)
- new net USB_DP1: U?.V14 (USB_DP1)
- new net USB_DP2: U?.W13 (USB_DP2)
- new net VDD: FB?.2, U?.G13 (VDD_PLL2), U?.J5 (VDD_PLL), U?.K6 (VDD), U?.L3 (VDD_ANA), U?.L5 (VDD), U?.L7 (VDD), U?.M6 (VDD), U?.M8 (VDD), U?.N1 (PDR_ON_CORE), U?.N2 (PDR_ON), U?.N5 (VDD), U?.N7 (VDD), U?.N9 (VDD), U?.P10 (VDD), U?.P6 (VDD), U?.P8 (VDD), U?.R11 (VDD), U?.R7 (VDD), U?.R9 (VDD)
- new net VDD_CORE: U?.E11 (VDDCORE), U?.E13 (VDDCORE), U?.E7 (VDDCORE), U?.E9 (VDDCORE), U?.F10 (VDDCORE), U?.F12 (VDDCORE), U?.F4 (VDDCORE), U?.F6 (VDDCORE), U?.F8 (VDDCORE), U?.G11 (VDDCORE), U?.G5 (VDDCORE), U?.G7 (VDDCORE), U?.G9 (VDDCORE), U?.H10 (VDDCORE), U?.H12 (VDDCORE), U?.H4 (VDDCORE), U?.H6 (VDDCORE), U?.H8 (VDDCORE), U?.J11 (VDDCORE), U?.J13 (VDDCORE), U?.J7 (VDDCORE), U?.J9 (VDDCORE), U?.K10 (VDDCORE), U?.K12 (VDDCORE), U?.K8 (VDDCORE), U?.L11 (VDDCORE), U?.L13 (VDDCORE), U?.L9 (VDDCORE), U?.M10 (VDDCORE), U?.M12 (VDDCORE), U?.N11 (VDDCORE), U?.N13 (VDDCORE), U?.P12 (VDDCORE), U?.R13 (VDDCORE)
- new net VDD_USB: U?.W12 (VDD3V3_USBHS), U?.W15 (VDD3V3_USBFS)

Commit message: update schematic and pdf
Parts:
- added C? (x2): 1u, Capacitor_SMD:C_0805_2012Metric, symbol Device:C_Small
- added C? (x6): 100n, Capacitor_SMD:C_0805_2012Metric, symbol Device:C_Small
- added R?: 240, Resistor_SMD:R_0805_2012Metric, symbol Device:R_Small
- added R? (x2): 1k, Resistor_SMD:R_0805_2012Metric, symbol Device:R_Small
- added unit 1 of U1
- added unit 2 of U1
- added unit 3 of U1
- added unit 4 of U1
- added unit 5 of U1
- added unit 6 of U1
- added unit 7 of U1
- added unit 8 of U1
- added Y? (x2): Crystal_Small, symbol Device:Crystal_Small
- gave numbers to parts that had none: 1
Connections:
- net GND: now also U1.T15 (BYPASS_REG1V8), C?.2, C?.2, C?.2, C?.2, C?.2, C?.2, C?.2, C?.2, R?.2, R?.2
- net VDD_USB: now also C?.1
- net DDR_DQ0: now reaches U1.A17 (DDR_DQ0)
- net DDR_DQ1: now reaches U1.A18 (DDR_DQ1)
- net DDR_DQ3: now reaches U1.B17 (DDR_DQ3)
- net DDR_DQ7: now reaches U1.B18 (DDR_DQ7)
- net DDR_~LDQS: now reaches U1.B19 (DDR_DQS0N)
- net DDR_LDM: now reaches U1.C18 (DDR_DQM0)
- net DDR_LDQS: now reaches U1.C19 (DDR_DQS0P)
- net DDR_DQ5: now reaches U1.D17 (DDR_DQ5)
- net DDR_DQ2: now reaches U1.D18 (DDR_DQ2)
- net DDR_DQ6: now reaches U1.D19 (DDR_DQ6)
- net VDD_DDR: now reaches U1.E15 (VDDQ_DDR)
- net VDD_DDR: now also U1.F14 (VDDQ_DDR), U1.G15 (VDDQ_DDR), U1.H14 (VDDQ_DDR), U1.J15 (VDDQ_DDR), U1.K14 (VDDQ_DDR), U1.L15 (VDDQ_DDR), U1.M14 (VDDQ_DDR), U1.N15 (VDDQ_DDR), U1.P14 (VDDQ_DDR), U1.R15 (VDDQ_DDR), R?.1
- net DDR_A7: now reaches U1.E17 (DDR_A7)
- net DDR_DQ4: now reaches U1.E18 (DDR_DQ4)
- net DDR_A13: now reaches U1.F17 (DDR_A13)
- net at U1.F18 (DDR_ZQ): now also R?.1
- net DDR_A3: now reaches U1.F19 (DDR_A3)
- net DDR_~RESET: now reaches U1.G16 (DDR_RESETN)
- net DDR_A9: now reaches U1.G17 (DDR_A9)
- net DDR_A2: now reaches U1.G18 (DDR_A2)
- net DDR_BA0: now reaches U1.G19 (DDR_BA0)
- net DDR_A5: now reaches U1.H17 (DDR_A5)
- net DDR_A0: now reaches U1.H18 (DDR_A0)
- net DDR_ODT: now reaches U1.H19 (DDR_ODT)
- net DDR_BA2: now reaches U1.J16 (DDR_BA2)
- net DDR_~WE: now reaches U1.J17 (DDR_WEN)
- net DDR_~CS: now reaches U1.J18 (DDR_CSN)
- net DDR_~CAS: now reaches U1.K17 (DDR_CASN)
- net DDR_~CK: now reaches U1.K19 (DDR_CLKN)
- net DDR_A15: now reaches U1.L16 (DDR_A15)
- net DDR_A12: now reaches U1.L17 (DDR_A12)
- net DDR_~RAS: now reaches U1.L18 (DDR_RASN)
- net DDR_CK: now reaches U1.L19 (DDR_CLKP)
- net DDR_A1: now reaches U1.M17 (DDR_A1)
- net DDR_A11: now reaches U1.M18 (DDR_A11)
- net DDR_A10: now reaches U1.M19 (DDR_A10)
- net DDR_A6: now reaches U1.N16 (DDR_A6)
- net DDR_BA1: now reaches U1.N17 (DDR_BA1)
- net DDR_A14: now reaches U1.N18 (DDR_A14)
- net DDR_A4: now reaches U1.P17 (DDR_A4)
- net DDR_DQ8: now reaches U1.P18 (DDR_DQ8)
- net DDR_CKE: now reaches U1.P19 (DDR_CKE)
- net DDR_A8: now reaches U1.R17 (DDR_A8)
- net DDR_DQ10: now reaches U1.R18 (DDR_DQ10)
- net DDR_DQ9: now reaches U1.T17 (DDR_DQ9)
- net DDR_DQ13: now reaches U1.T18 (DDR_DQ13)
- net DDR_~UDQS: now reaches U1.T19 (DDR_DQS1N)
- net DDR_UDM: now reaches U1.U18 (DDR_DQM1)
- net DDR_UDQS: now reaches U1.U19 (DDR_DQS1P)
- net DDR_DQ14: now reaches U1.V18 (DDR_DQ14)
- net DDR_DQ11: now reaches U1.V19 (DDR_DQ11)
- net at U1.W16 (DDR_VREF): now also C?.1, R?.1, R?.2
- net DDR_DQ15: now reaches U1.W17 (DDR_DQ15)
- net DDR_DQ12: now reaches U1.W18 (DDR_DQ12)
- net VDDA1V8_REG: now reaches U1.V11 (VDDA1V8_REG)
- net VDDA1V8_REG: now also C?.1
- net at U1.W11 (VDDA1V1_REG): now also C?.1
- net CPU_JTMS-SWDCLK renamed CPU_SWCLK
- net CPU_JTMS-SWDIO renamed CPU_SWDIO
- net CPU_JTMS-TRACESW0 renamed CPU_SWO
- new net: C?.1, U1.H2 (PC15-OSC32_OUT), Y?.1
- new net: C?.1, U1.H1 (PC14-OSC32_IN), Y?.2
- new net: C?.1, U1.M2 (PH1-OSC_OUT), Y?.1
- new net: C?.1, U1.M1 (PH0-OSC_IN), Y?.2
- new net DEBUG_UART4_RX: U1.T13 (PB2)
- new net DEBUG_UART4_TX: U1.V6 (PG11)
- new net ETH1_MDC: U1.V2 (PC1)
- new net ETH1_MDIO: U1.W2 (PA2)
- new net ETH1_RMII_CRS_DV: U1.T6 (PA7)
- new net ETH1_RMII_REF_CLK: U1.U4 (PA1)
- new net ETH1_RMII_RXD0: U1.W4 (PC4)
- new net ETH1_RMII_RXD1: U1.V4 (PC5)
- new net ETH1_RMII_TXD0: U1.V5 (PB12)
- new net ETH1_RMII_TXD1: U1.T9 (PB13)
- new net ETH1_RMII_TX_EN: U1.V1 (PB11)
- new net ETH_INTRP: U1.T5 (PA6)
- new net SDMMC1_CK: U1.C10 (PC12)
- new net SDMMC1_CMD: U1.B10 (PD2)
- new net SDMMC1_D0: U1.C11 (PC8)
- new net SDMMC1_D1: U1.A10 (PC9)
- new net SDMMC1_D2: U1.D11 (PC10)
- new net SDMMC1_D3: U1.A11 (PC11)
- new net SDMMC1_DET: U1.B5 (PB7)
- no-connect marks 0 -> 3
Other:
- moved on the sheet: C?, D?, FB?, R?, U1M, U1N
